Commit message: sim

File: shooter/urdf/shooter.urdf.xacro (robot description, xacro)
@@ -3,4 +3,5 @@
   <!-- Parameters -->
   <xacro:arg name="use_sim" default="false"/>
+  <xacro:property name="use_sim" value="$(arg use_sim)"/>
   <!-- Properties -->
   <xacro:property name="wheel_radius" value="0.05"/>
@@ -119,27 +120,71 @@
     <origin xyz="${-base_length/2 + wheel_radius/2} 0 ${-wheel_radius/2}" rpy="0 0 0"/>
   </joint>
-  <!-- ros2_control -->
-  <ros2_control name="epos_system" type="system">
-    <hardware>
-      <plugin>epos/EPOSHardwareInterface</plugin>
-      <param name="device_name">EPOS4</param>
-      <param name="protocol_stack_name">MAXON SERIAL V2</param>
-      <param name="interface_name">USB</param>
-      <param name="port_name">USB0</param>
-      <param name="baudrate">1000000</param>
-      <param name="counts_per_revolution">4096</param>
-    </hardware>
-    <joint name="left_wheel_joint">
-      <param name="node_id">1</param>
-      <command_interface name="velocity"/>
-      <state_interface name="position"/>
-      <state_interface name="velocity"/>
-    </joint>
-    <joint name="right_wheel_joint">
-      <param name="node_id">2</param>
-      <command_interface name="velocity"/>
-      <state_interface name="position"/>
-      <state_interface name="velocity"/>
-    </joint>
-  </ros2_control>
+  <!-- ros2_control - Real Hardware -->
+  <xacro:unless value="${use_sim}">
+    <ros2_control name="epos_system" type="system">
+      <hardware>
+        <plugin>epos/EPOSHardwareInterface</plugin>
+        <param name="device_name">EPOS4</param>
+        <param name="protocol_stack_name">MAXON SERIAL V2</param>
+        <param name="interface_name">USB</param>
+        <param name="port_name">USB0</param>
+        <param name="baudrate">1000000</param>
+        <param name="counts_per_revolution">4096</param>
+      </hardware>
+      <joint name="left_wheel_joint">
+        <param name="node_id">1</param>
+        <command_interface name="velocity"/>
+        <state_interface name="position"/>
+        <state_interface name="velocity"/>
+      </joint>
+      <joint name="right_wheel_joint">
+        <param name="node_id">2</param>
+        <command_interface name="velocity"/>
+        <state_interface name="position"/>
+        <state_interface name="velocity"/>
+      </joint>
+    </ros2_control>
+  </xacro:unless>
+  <!-- ros2_control - Gazebo Simulation -->
+  <xacro:if value="${use_sim}">
+    <ros2_control name="GazeboSystem" type="system">
+      <hardware>
+        <plugin>gz_ros2_control/GazeboSimSystem</plugin>
+      </hardware>
+      <joint name="left_wheel_joint">
+        <command_interface name="velocity"/>
+        <state_interface name="position"/>
+        <state_interface name="velocity"/>
+      </joint>
+      <joint name="right_wheel_joint">
+        <command_interface name="velocity"/>
+        <state_interface name="position"/>
+        <state_interface name="velocity"/>
+      </joint>
+    </ros2_control>
+    <!-- Gazebo plugins -->
+    <gazebo>
+      <plugin filename="gz_ros2_control-system" name="gz_ros2_control::GazeboSimROS2ControlPlugin">
+        <parameters>$(find shooter)/config/controllers.yaml</parameters>
+      </plugin>
+    </gazebo>
+    <!-- Wheel friction -->
+    <gazebo reference="left_wheel">
+      <mu1>1.0</mu1>
+      <mu2>1.0</mu2>
+      <kp>1000000.0</kp>
+      <kd>100.0</kd>
+    </gazebo>
+    <gazebo reference="right_wheel">
+      <mu1>1.0</mu1>
+      <mu2>1.0</mu2>
+      <kp>1000000.0</kp>
+      <kd>100.0</kd>
+    </gazebo>
+    <!-- Caster wheel - low friction for sliding -->
+    <gazebo reference="caster_wheel">
+      <mu1>0.001</mu1>
+      <mu2>0.001</mu2>
+    </gazebo>
+  </xacro:if>
 </robot>

Commit message: yolo v4 tin

File: shooter/urdf/shooter.urdf.xacro (robot description, xacro)
@@ -8,4 +8,5 @@
   <xacro:property name="wheel_width" value="0.04"/>
   <xacro:property name="wheel_separation" value="0.3"/>
+  <xacro:property name="wheelbase" value="0.25"/>
   <xacro:property name="base_length" value="0.4"/>
   <xacro:property name="base_width" value="0.3"/>
@@ -49,74 +50,55 @@
     <origin xyz="0 0 ${base_height/2}" rpy="0 0 0"/>
   </joint>
-  <!-- Left Wheel -->
-  <link name="left_wheel">
-    <visual>
-      <geometry>
-        <cylinder radius="${wheel_radius}" length="${wheel_width}"/>
-      </geometry>
-      <material name="black"/>
-    </visual>
-    <collision>
-      <geometry>
-        <cylinder radius="${wheel_radius}" length="${wheel_width}"/>
-      </geometry>
-    </collision>
-    <inertial>
-      <mass value="0.5"/>
-      <inertia ixx="0.001" ixy="0" ixz="0" iyy="0.001" iyz="0" izz="0.001"/>
-    </inertial>
-  </link>
-  <joint name="left_wheel_joint" type="continuous">
+  <!-- Wheel Macro -->
+  <xacro:macro name="wheel" params="name">
+    <link name="${name}">
+      <visual>
+        <geometry>
+          <cylinder radius="${wheel_radius}" length="${wheel_width}"/>
+        </geometry>
+        <material name="black"/>
+      </visual>
+      <collision>
+        <geometry>
+          <cylinder radius="${wheel_radius}" length="${wheel_width}"/>
+        </geometry>
+      </collision>
+      <inertial>
+        <mass value="0.5"/>
+        <inertia ixx="0.001" ixy="0" ixz="0" iyy="0.001" iyz="0" izz="0.001"/>
+      </inertial>
+    </link>
+  </xacro:macro>
+  <!-- Front Left Wheel -->
+  <xacro:wheel name="front_left_wheel"/>
+  <joint name="front_left_wheel_joint" type="continuous">
     <parent link="base_link"/>
-    <child link="left_wheel"/>
-    <origin xyz="0 ${wheel_separation/2} 0" rpy="${-pi/2} 0 0"/>
+    <child link="front_left_wheel"/>
+    <origin xyz="${wheelbase/2} ${wheel_separation/2} 0" rpy="${-pi/2} 0 0"/>
     <axis xyz="0 0 1"/>
   </joint>
-  <!-- Right Wheel -->
-  <link name="right_wheel">
-    <visual>
-      <geometry>
-        <cylinder radius="${wheel_radius}" length="${wheel_width}"/>
-      </geometry>
-      <material name="black"/>
-    </visual>
-    <collision>
-      <geometry>
-        <cylinder radius="${wheel_radius}" length="${wheel_width}"/>
-      </geometry>
-    </collision>
-    <inertial>
-      <mass value="0.5"/>
-      <inertia ixx="0.001" ixy="0" ixz="0" iyy="0.001" iyz="0" izz="0.001"/>
-    </inertial>
-  </link>
-  <joint name="right_wheel_joint" type="continuous">
+  <!-- Rear Left Wheel -->
+  <xacro:wheel name="rear_left_wheel"/>
+  <joint name="rear_left_wheel_joint" type="continuous">
     <parent link="base_link"/>
-    <child link="right_wheel"/>
-    <origin xyz="0 ${-wheel_separation/2} 0" rpy="${-pi/2} 0 0"/>
+    <child link="rear_left_wheel"/>
+    <origin xyz="${-wheelbase/2} ${wheel_separation/2} 0" rpy="${-pi/2} 0 0"/>
     <axis xyz="0 0 1"/>
   </joint>
-  <!-- Caster Wheel (for stability) -->
-  <link name="caster_wheel">
-    <visual>
-      <geometry>
-        <sphere radius="${wheel_radius/2}"/>
-      </geometry>
-      <material name="black"/>
-    </visual>
-    <collision>
-      <geometry>
-        <sphere radius="${wheel_radius/2}"/>
-      </geometry>
-    </collision>
-    <inertial>
-      <mass value="0.1"/>
-      <inertia ixx="0.0001" ixy="0" ixz="0" iyy="0.0001" iyz="0" izz="0.0001"/>
-    </inertial>
-  </link>
-  <joint name="caster_wheel_joint" type="fixed">
+  <!-- Front Right Wheel -->
+  <xacro:wheel name="front_right_wheel"/>
+  <joint name="front_right_wheel_joint" type="continuous">
     <parent link="base_link"/>
-    <child link="caster_wheel"/>
-    <origin xyz="${-base_length/2 + wheel_radius/2} 0 ${-wheel_radius/2}" rpy="0 0 0"/>
+    <child link="front_right_wheel"/>
+    <origin xyz="${wheelbase/2} ${-wheel_separation/2} 0" rpy="${-pi/2} 0 0"/>
+    <axis xyz="0 0 1"/>
+  </joint>
+  <!-- Rear Right Wheel -->
+  <xacro:wheel name="rear_right_wheel"/>
+  <joint name="rear_right_wheel_joint" type="continuous">
+    <parent link="base_link"/>
+    <child link="rear_right_wheel"/>
+    <origin xyz="${-wheelbase/2} ${-wheel_separation/2} 0" rpy="${-pi/2} 0 0"/>
+    <axis xyz="0 0 1"/>
   </joint>
   <!-- ros2_control - Real Hardware -->
@@ -132,5 +114,5 @@
         <param name="counts_per_revolution">4096</param>
       </hardware>
-      <joint name="left_wheel_joint">
+      <joint name="front_left_wheel_joint">
         <param name="node_id">1</param>
         <command_interface name="velocity"/>
@@ -138,5 +120,5 @@
         <state_interface name="velocity"/>
       </joint>
-      <joint name="right_wheel_joint">
+      <joint name="front_right_wheel_joint">
         <param name="node_id">2</param>
         <command_interface name="velocity"/>
@@ -152,10 +134,20 @@
         <plugin>gz_ros2_control/GazeboSimSystem</plugin>
       </hardware>
-      <joint name="left_wheel_joint">
+      <joint name="front_left_wheel_joint">
         <command_interface name="velocity"/>
         <state_interface name="position"/>
         <state_interface name="velocity"/>
       </joint>
-      <joint name="right_wheel_joint">
+      <joint name="rear_left_wheel_joint">
+        <command_interface name="velocity"/>
+        <state_interface name="position"/>
+        <state_interface name="velocity"/>
+      </joint>
+      <joint name="front_right_wheel_joint">
+        <command_interface name="velocity"/>
+        <state_interface name="position"/>
+        <state_interface name="velocity"/>
+      </joint>
+      <joint name="rear_right_wheel_joint">
         <command_interface name="velocity"/>
         <state_interface name="position"/>
@@ -170,5 +162,5 @@
     </gazebo>
     <!-- Wheel friction -->
-    <gazebo reference="left_wheel">
+    <gazebo reference="front_left_wheel">
       <mu1>1.0</mu1>
       <mu2>1.0</mu2>
@@ -176,5 +168,5 @@
       <kd>100.0</kd>
     </gazebo>
-    <gazebo reference="right_wheel">
+    <gazebo reference="rear_left_wheel">
       <mu1>1.0</mu1>
       <mu2>1.0</mu2>
@@ -182,8 +174,15 @@
       <kd>100.0</kd>
     </gazebo>
-    <!-- Caster wheel - low friction for sliding -->
-    <gazebo reference="caster_wheel">
-      <mu1>0.001</mu1>
-      <mu2>0.001</mu2>
+    <gazebo reference="front_right_wheel">
+      <mu1>1.0</mu1>
+      <mu2>1.0</mu2>
+      <kp>1000000.0</kp>
+      <kd>100.0</kd>
+    </gazebo>
+    <gazebo reference="rear_right_wheel">
+      <mu1>1.0</mu1>
+      <mu2>1.0</mu2>
+      <kp>1000000.0</kp>
+      <kd>100.0</kd>
     </gazebo>
   </xacro:if>

Commit message: 実機で動作確認

File: shooter/urdf/shooter.urdf.xacro (robot description, xacro)
@@ -3,5 +3,7 @@
   <!-- Parameters -->
   <xacro:arg name="use_sim" default="false"/>
+  <xacro:arg name="usb_port" default="USB0"/>
   <xacro:property name="use_sim" value="$(arg use_sim)"/>
+  <xacro:property name="usb_port" value="$(arg usb_port)"/>
   <!-- Properties -->
   <xacro:property name="wheel_radius" value="0.05"/>
@@ -110,10 +112,10 @@
         <param name="protocol_stack_name">MAXON SERIAL V2</param>
         <param name="interface_name">USB</param>
-        <param name="port_name">USB0</param>
+        <param name="port_name">${usb_port}</param>
         <param name="baudrate">1000000</param>
         <param name="counts_per_revolution">4096</param>
       </hardware>
       <joint name="front_left_wheel_joint">
-        <param name="node_id">1</param>
+        <param name="node_id">2</param>
         <command_interface name="velocity"/>
         <state_interface name="position"/>
@@ -121,5 +123,5 @@
       </joint>
       <joint name="front_right_wheel_joint">
-        <param name="node_id">2</param>
+        <param name="node_id">1</param>
         <command_interface name="velocity"/>
         <state_interface name="position"/>

Commit message: 位置制御・ホーミングモード

File: shooter/urdf/shooter.urdf.xacro (robot description, xacro)
@@ -104,4 +104,53 @@
     <axis xyz="0 0 1"/>
   </joint>
+  <!-- Pan-Tilt Mechanism -->
+  <link name="pan_link">
+    <visual>
+      <geometry>
+        <cylinder radius="0.03" length="0.05"/>
+      </geometry>
+      <material name="white"/>
+    </visual>
+    <collision>
+      <geometry>
+        <cylinder radius="0.03" length="0.05"/>
+      </geometry>
+    </collision>
+    <inertial>
+      <mass value="0.2"/>
+      <inertia ixx="0.0001" ixy="0" ixz="0" iyy="0.0001" iyz="0" izz="0.0001"/>
+    </inertial>
+  </link>
+  <joint name="pan_joint" type="revolute">
+    <parent link="chassis"/>
+    <child link="pan_link"/>
+    <origin xyz="0 0 ${base_height/2 + 0.025}" rpy="0 0 0"/>
+    <axis xyz="0 0 1"/>
+    <limit lower="${-pi}" upper="${pi}" effort="10" velocity="3.14"/>
+  </joint>
+  <link name="tilt_link">
+    <visual>
+      <geometry>
+        <box size="0.05 0.08 0.03"/>
+      </geometry>
+      <material name="black"/>
+    </visual>
+    <collision>
+      <geometry>
+        <box size="0.05 0.08 0.03"/>
+      </geometry>
+    </collision>
+    <inertial>
+      <mass value="0.1"/>
+      <inertia ixx="0.0001" ixy="0" ixz="0" iyy="0.0001" iyz="0" izz="0.0001"/>
+    </inertial>
+  </link>
+  <joint name="tilt_joint" type="revolute">
+    <parent link="pan_link"/>
+    <child link="tilt_link"/>
+    <origin xyz="0 0 0.04" rpy="0 0 0"/>
+    <axis xyz="0 1 0"/>
+    <limit lower="${-pi/2}" upper="${pi/2}" effort="10" velocity="3.14"/>
+  </joint>
   <!-- ros2_control - Real Hardware -->
   <xacro:unless value="${use_sim}">
@@ -116,4 +165,11 @@
         <param name="counts_per_revolution">4096</param>
       </hardware>
+      <!-- Velocity control joints (node_id 1, 2) -->
+      <joint name="front_right_wheel_joint">
+        <param name="node_id">1</param>
+        <command_interface name="velocity"/>
+        <state_interface name="position"/>
+        <state_interface name="velocity"/>
+      </joint>
       <joint name="front_left_wheel_joint">
         <param name="node_id">2</param>
@@ -122,7 +178,14 @@
         <state_interface name="velocity"/>
       </joint>
-      <joint name="front_right_wheel_joint">
-        <param name="node_id">1</param>
-        <command_interface name="velocity"/>
+      <!-- Position control joints (node_id 3, 4) -->
+      <joint name="pan_joint">
+        <param name="node_id">3</param>
+        <command_interface name="position"/>
+        <state_interface name="position"/>
+        <state_interface name="velocity"/>
+      </joint>
+      <joint name="tilt_joint">
+        <param name="node_id">4</param>
+        <command_interface name="position"/>
         <state_interface name="position"/>
         <state_interface name="velocity"/>
