Commit message: Update

File: shooter_bringup/urdf/shooter_ros2_control.urdf.xacro (robot description, xacro)
@@ -25,22 +25,27 @@
       <state_interface name="velocity"/>
     </joint>
-    <!-- Position control joints (node_id 3, 4) -->
+    <!-- Velocity control joints (node_id 3, 4) -->
     <!-- Pan joint: counts_per_revolution calculated from homing offset (1650000 counts ≈ 90°) -->
     <joint name="pan_joint">
       <param name="node_id">3</param>
       <param name="counts_per_revolution">6600000</param>
-      <command_interface name="position"/>
+      <command_interface name="velocity"/>
       <state_interface name="position"/>
       <state_interface name="velocity"/>
     </joint>
-    <!-- tilt_joint temporarily disabled
     <joint name="tilt_joint">
       <param name="node_id">4</param>
       <param name="counts_per_revolution">6600000</param>
-      <command_interface name="position"/>
+      <command_interface name="velocity"/>
       <state_interface name="position"/>
       <state_interface name="velocity"/>
     </joint>
-    -->
+    <!-- Shooter motor (node_id 5) - velocity control -->
+    <joint name="shooter_joint">
+      <param name="node_id">5</param>
+      <command_interface name="velocity"/>
+      <state_interface name="position"/>
+      <state_interface name="velocity"/>
+    </joint>
   </ros2_control>
 </robot>
