Commit message: Refactoring

File: chikurin_description/urdf/chikurin.urdf.xacro (robot description, xacro)
@@ -1,4 +1,4 @@
 <?xml version="1.0"?>
-<robot xmlns:xacro="http://www.ros.org/wiki/xacro" name="shooter">
+<robot xmlns:xacro="http://www.ros.org/wiki/xacro" name="chikurin">
   <!-- Parameters -->
   <xacro:arg name="use_sim" default="false"/>
@@ -155,8 +155,8 @@
   <!-- ros2_control configuration (conditional include) -->
   <xacro:if value="${use_sim}">
-    <xacro:include filename="$(find shooter_simulation)/urdf/shooter_gazebo.urdf.xacro"/>
+    <xacro:include filename="$(find chikurin_description)/urdf/gazebo.urdf.xacro"/>
   </xacro:if>
   <xacro:unless value="${use_sim}">
-    <xacro:include filename="$(find shooter_bringup)/urdf/shooter_ros2_control.urdf.xacro"/>
+    <xacro:include filename="$(find chikurin_description)/urdf/ros2_control.urdf.xacro"/>
   </xacro:unless>
 </robot>

File: chikurin_description/urdf/gazebo.urdf.xacro (robot description, xacro)
@@ -26,9 +26,20 @@
       <state_interface name="velocity"/>
     </joint>
+    <!-- Pan-Tilt joints -->
+    <joint name="pan_joint">
+      <command_interface name="velocity"/>
+      <state_interface name="position"/>
+      <state_interface name="velocity"/>
+    </joint>
+    <joint name="tilt_joint">
+      <command_interface name="velocity"/>
+      <state_interface name="position"/>
+      <state_interface name="velocity"/>
+    </joint>
   </ros2_control>
   <!-- Gazebo ros2_control plugin -->
   <gazebo>
     <plugin filename="gz_ros2_control-system" name="gz_ros2_control::GazeboSimROS2ControlPlugin">
-      <parameters>$(find shooter_simulation)/config/sim_controllers.yaml</parameters>
+      <parameters>$(find chikurin_description)/config/sim_controllers.yaml</parameters>
     </plugin>
   </gazebo>
